File: eeg schematic/eeg.kicad_sch (KiCad schematic)
At the start: 21 parts, among them IC1 INA121PA, J1 Conn_01x02_Pin, U1 LF353P, U2 LF353P

Commit message: component values for schematic
Parts:
- removed J1: Conn_01x02_Pin, symbol Connector:Conn_01x02_Pin
- added C6, C7: 100nF, symbol Device:C
- added R13, R14, R15: 110kR, symbol Device:R
- C1, C2, C4, C5: value C -> 100nF
- C3: value C -> 1uF
- R1: value R -> 5R
- R10, R11: value R -> 33kR
- R12: value R -> 1kR
- R2, R3: value R -> 2kR
- R4: value R -> 1.6MR
- R5, R9: value R -> 110kR
- R6, R7, R8: value R -> 10kR
Connections:
- net +9V: now also C6.1
- net GND: now also C6.2, C7.2
- net RL Drive: now also R13.2; no longer U1.1 (1OUT), U1.2 (1IN-)
- net at C2.1, IC1.5 (REF), R2.2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: now also C7.1
- net at IC1.2 (V-IN): now also R14.2
- net at IC1.3 (V+IN): now also R15.2
- new net: R13.1, U1.1 (1OUT), U1.2 (1IN-)
- new net V+: R15.1
- new net V-: R14.1
Other:
- note added: "gain = 10000 typ. input = 10-100 uV"
